File: eagle/HHV_SCA_Demo-P1.brd (EAGLE design)
At the start: 72.8 x 53.8 mm, 35 parts, among them CN1 MINIUSB-SMD, CN3 CON, U1 PIC12F1572, U2 FT230XS, U3 AOZ8105CI

Commit message: eagle: Final draft of P1 rev
Parts:
- removed FB2: (no value), rcl:R0603
- removed LED1, LED2, LED3, LED4: (no value), led:LED3MM
- added D1, D2, D3, D4: (no value), led:LED3MM
- moved U$1 81.2 mm to (14.0, 32.0), flipped to the bottom
- moved C3 60.4 mm to (70.2, 36.2), turned to 90 degrees
- moved R8 58.1 mm to (60.9, 31.4), turned to 180 degrees
- moved U3 56.0 mm to (63.0, 40.6), turned to 180 degrees
- moved CN1 55.6 mm to (64.8, 48.3)
- moved R7 53.4 mm to (65.0, 31.4)
- moved C2 53.4 mm to (68.5, 36.2), turned to 90 degrees
- moved C5 52.6 mm to (68.5, 32.6), turned to 270 degrees
- moved FB1 52.2 mm to (66.0, 39.9), turned to 90 degrees
- moved U2 43.0 mm to (63.0, 35.1), turned to 0 degrees
- moved SJ1 32.7 mm to (52.6, 35.1), turned to 0 degrees
- moved SJ2 32.0 mm to (52.6, 37.8), turned to 0 degrees
- moved R9 30.7 mm to (71.1, 27.1), turned to 90 degrees
- moved R5 28.6 mm to (35.7, 47.4), turned to 0 degrees
- moved R6 26.1 mm to (30.0, 47.4), turned to 0 degrees
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Connections:
- removed net ICSPDAT: CN3.4
- removed net N$10: C3.1
- removed net N$7: CN1.VSS, FB2.2
- removed net N$9: C3.2
- net 3V3: now also D1.A, D2.A, D3.A, D4.A; no longer LED1.A, LED2.A, LED3.A, LED4.A
- net FTDI_RXD: now also CN3.4
- net N$11: now also D3.K; no longer LED3.K
- net N$13: now also D4.K; no longer LED4.K
- net N$3: now also D2.K; no longer LED2.K
- net N$8: now also D1.K; no longer LED1.K
- net USB_5V: now also C3.1
- net USB_DM: now also U3.1; no longer U3.6
- net USB_DP: now also U3.3; no longer U3.1
- net VSS: now also C3.2, CN1.VSS; no longer FB2.1
Routing:
- net 3V3: track 0.00 -> 142.1 mm, vias 0 -> 3
- net AN2: track 0.00 -> 63.9 mm, vias 0 -> 1
- net MCLR#: track 0.00 -> 45.4 mm, vias 0 -> 2
- net LED_G#: track 0.00 -> 33.3 mm
- net LED_R#: track 0.00 -> 27.3 mm
- net N$5: track 0.00 -> 25.4 mm
- net N$2: track 0.00 -> 25.4 mm
- net FTDI_RXD: track 0.00 -> 24.3 mm
- net USB_5V: track 0.00 -> 20.2 mm, vias 0 -> 2
- net FTDI_TXD: track 0.00 -> 20.0 mm
- net USB_DM: track 0.00 -> 16.0 mm
- net USB_DP: track 0.00 -> 16.0 mm
- net LED_RXD#: track 0.00 -> 14.3 mm, vias 0 -> 2
- net VSS: track 0.00 -> 13.6 mm, vias 0 -> 12
- net LED_TXD#: track 0.00 -> 11.3 mm, vias 0 -> 2
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- added copper zone on layer 1, net VSS
- added copper zone on layer 16, net VSS
Other:
- board text added: "0"
- board text added: "1"
- board text added: "2"
- board text added: "3"
- board text added: "C1"
- board text added: "C2"
- board text added: "C3"
- board text added: "C4"
- board text added: "C5"
- board text added: "CN1"
- board text added: "CN2"
- board text added: "CN3"
- board text added: "Connect USB to host Connect USB AX PRO Analyzer Open USB serial terminal on host Follow on-screen instructions"
- board text added: "Cut when ICSP Short for operation"
- board text added: "D1"
- board text added: "D2"
- board text added: "D3"
- board text added: "D4"
- board text added: "DEF CON HHV Side Channel Timing Attack Demo"
- board text added: "FB1"
- board text added: "Green"
- board text added: "HHV SCA Rev P1"
- board text added: "R1"
- board text added: "R10"
- board text added: "R2"
- board text added: "R3"
- board text added: "R4"
- board text added: "R5"
- board text added: "R6"
- board text added: "R7"
- board text added: "R8"
- board text added: "R9"
- board text added: "RX"
- board text added: "Red"
- board text added: "Reset"
- board text added: "SW1"
- board text added: "SW2"
- board text added: "SW3"
- board text added: "SW4"
- board text added: "SW5"
- board text added: "TX"
- board text added: "U1"
- board text added: "U2"
- board text added: "U3"
- board text added: "USBee AX PRO"

Commit message: eagle: Finalized schematic and board files
Added donation text to back silkscreen
Changed schematic names of S* to SW*
Removed value from SW5
Added color values to D*
Parts:
- D1, D4: value (none) -> GRN
- D2, D3: value (none) -> RED
- SW5: value 3 -> (none)
- renumbered S1 to SW1, S2 to SW2, S3 to SW3, S4 to SW4, S5 to SW5
Other:
- board text added: "PCBs donated to the HHV by OSHPark Design, components, & assembly donated by KBEmbedded"
Changed lines of the file:
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@@
 <text x="15.748" y="36.32708125" size="0.8128" layer="38" font="vector" rot="MR0">www.KBEmbedded.com</text>
 <text x="14.351" y="30.734" size="0.8128" layer="38" font="vector" rot="MR0">HHV SCA Rev P1</text>
-<text x="57.912" y="2.159" size="1.778" layer="38" font="vector" ratio="20" rot="MR0">Connect USB to host
+<text x="60.579" y="2.286" size="1.778" layer="38" font="vector" ratio="20" rot="MR0">Connect USB to host
 Connect USB AX PRO Analyzer
 Open USB serial terminal on host
 Follow on-screen instructions</text>
+<text x="55.499" y="42.164" size="0.8128" layer="38" font="vector" rot="MR0">PCBs donated to the HHV by OSHPark
+Design, components, &amp; assembly donated by KBEmbedded</text>
 </plain>
 <attributes>
@@
 <attribute name="OC_FARNELL" value="unknown" x="47.5" y="52.152" size="1.778" layer="27" rot="R180" display="off"/>
 </element>
-<element name="S1" library="switch-omron" package="B3F-10XX" value="" x="9.525" y="15.875" rot="R180">
+<element name="SW1" library="switch-omron" package="B3F-10XX" value="" x="9.525" y="15.875" rot="R180">
 <attribute name="OC_NEWARK" value="36M3542" x="9.525" y="15.875" size="1.778" layer="27" rot="R180" display="off"/>
 <attribute name="MPN" value="B3F-1000" x="9.525" y="15.875" size="1.778" layer="27" rot="R180" display="off"/>
@@
 <attribute name="OC_FARNELL" value="176432" x="9.525" y="15.875" size="1.778" layer="27" rot="R180" display="off"/>
 </element>
-<element name="S2" library="switch-omron" package="B3F-10XX" value="" x="27.305" y="15.875" rot="R180">
+<element name="SW2" library="switch-omron" package="B3F-10XX" value="" x="27.305" y="15.875" rot="R180">
 <attribute name="OC_NEWARK" value="36M3542" x="27.305" y="15.875" size="1.778" layer="27" rot="R180" display="off"/>
 <attribute name="MPN" value="B3F-1000" x="27.305" y="15.875" size="1.778" layer="27" rot="R180" display="off"/>
@@
 <attribute name="OC_FARNELL" value="176432" x="27.305" y="15.875" size="1.778" layer="27" rot="R180" display="off"/>
 </element>
-<element name="S3" library="switch-omron" package="B3F-10XX" value="" x="45.085" y="15.875" rot="R180">
+<element name="SW3" library="switch-omron" package="B3F-10XX" value="" x="45.085" y="15.875" rot="R180">
 <attribute name="OC_NEWARK" value="36M3542" x="45.085" y="15.875" size="1.778" layer="27" rot="R180" display="off"/>
 <attribute name="MPN" value="B3F-1000" x="45.085" y="15.875" size="1.778" layer="27" rot="R180" display="off"/>
@@
 <attribute name="OC_FARNELL" value="176432" x="45.085" y="15.875" size="1.778" layer="27" rot="R180" display="off"/>
 </element>
-<element name="S4" library="switch-omron" package="B3F-10XX" value="" x="62.865" y="15.875" rot="R180">
+<element name="SW4" library="switch-omron" package="B3F-10XX" value="" x="62.865" y="15.875" rot="R180">
 <attribute name="OC_NEWARK" value="36M3542" x="62.865" y="15.875" size="1.778" layer="27" rot="R180" display="off"/>
 <attribute name="MPN" value="B3F-1000" x="62.865" y="15.875" size="1.778" layer="27" rot="R180" display="off"/>
@@
 <element name="C4" library="rcl" package="C0603K" value="10nF" x="66.929" y="42.545"/>
 <element name="C5" library="rcl" package="C0603K" value=".1uF" x="68.453" y="32.639" rot="R270"/>
-<element name="D3" library="led" package="LED3MM" value="" x="68.072" y="27.051"/>
-<element name="D4" library="led" package="LED3MM" value="" x="59.944" y="27.051"/>
+<element name="D3" library="led" package="LED3MM" value="RED" x="68.072" y="27.051"/>
+<element name="D4" library="led" package="LED3MM" value="GRN" x="59.944" y="27.051"/>
 <element name="R9" library="rcl" package="R0603" value="100" x="71.12" y="27.051" rot="R90"/>
 <element name="R10" library="rcl" package="R0603" value="100" x="62.992" y="27.051" rot="R90"/>
-<element name="D1" library="led" package="LED3MM" value="" x="35.687" y="50.927" rot="R270"/>
-<element name="D2" library="led" package="LED3MM" value="" x="29.972" y="50.927" rot="R270"/>
+<element name="D1" library="led" package="LED3MM" value="GRN" x="35.687" y="50.927" rot="R270"/>
+<element name="D2" library="led" package="LED3MM" value="RED" x="29.972" y="50.927" rot="R270"/>
 <element name="CN2" library="con-lstb" package="MA05-2" value="" x="19.304" y="49.276" rot="R180">
 <attribute name="OC_NEWARK" value="unknown" x="19.304" y="49.276" size="1.778" layer="27" rot="R180" display="off"/>
@@
 </element>
 <element name="U1" library="cuslibrary" package="DIL8" value="PIC12F1572" x="44.196" y="36.449"/>
-<element name="S5" library="switch-omron" package="B3F-10XX" value="3" x="31.496" y="36.449">
+<element name="SW5" library="switch-omron" package="B3F-10XX" value="" x="31.496" y="36.449">
 <attribute name="OC_NEWARK" value="36M3542" x="31.496" y="36.449" size="1.778" layer="27" display="off"/>
 <attribute name="MPN" value="B3F-1000" x="31.496" y="36.449" size="1.778" layer="27" display="off"/>
@@
 <contactref element="CN3" pad="1"/>
 <contactref element="U1" pad="4"/>
-<contactref element="S5" pad="4"/>
-<contactref element="S5" pad="3"/>
+<contactref element="SW5" pad="4"/>
+<contactref element="SW5" pad="3"/>
 <wire x1="48.006" y1="32.639" x2="46.228" y2="30.861" width="0.254" layer="1"/>
 <wire x1="46.228" y1="30.861" x2="42.545" y2="30.861" width="0.254" layer="1"/>
@@
 <signal name="VSS">
 <contactref element="CN3" pad="3"/>
-<contactref element="S4" pad="2"/>
-<contactref element="S4" pad="1"/>
-<contactref element="S3" pad="2"/>
-<contactref element="S3" pad="1"/>
-<contactref element="S2" pad="2"/>
-<contactref element="S2" pad="1"/>
-<contactref element="S1" pad="2"/>
-<contactref element="S1" pad="1"/>
+<contactref element="SW4" pad="2"/>
+<contactref element="SW4" pad="1"/>
+<contactref element="SW3" pad="2"/>
+<contactref element="SW3" pad="1"/>
+<contactref element="SW2" pad="2"/>
+<contactref element="SW2" pad="1"/>
+<contactref element="SW1" pad="2"/>
+<contactref element="SW1" pad="1"/>
 <contactref element="U2" pad="13"/>
 <contactref element="U2" pad="5"/>
@@
 <contactref element="CN2" pad="10"/>
 <contactref element="U1" pad="8"/>
-<contactref element="S5" pad="1"/>
-<contactref element="S5" pad="2"/>
+<contactref element="SW5" pad="1"/>
+<contactref element="SW5" pad="2"/>
 <contactref element="C1" pad="2"/>
 <polygon width="0.254" layer="16">
@@
 </signal>
 <signal name="N$1">
-<contactref element="S4" pad="4"/>
-<contactref element="S4" pad="3"/>
+<contactref element="SW4" pad="4"/>
+<contactref element="SW4" pad="3"/>
 <contactref element="R4" pad="1"/>
 <wire x1="66.1162" y1="18.1356" x2="63.754" y2="18.1356" width="0.254" layer="1"/>
@@
 <signal name="N$2">
 <contactref element="R4" pad="2"/>
-<contactref element="S3" pad="4"/>
-<contactref element="S3" pad="3"/>
+<contactref element="SW3" pad="4"/>
+<contactref element="SW3" pad="3"/>
 <contactref element="R3" pad="1"/>
 <wire x1="62.015" y1="20.955" x2="45.935" y2="20.955" width="0.254" layer="1"/>
@@
 <signal name="N$5">
 <contactref element="R3" pad="2"/>
-<contactref element="S2" pad="4"/>
-<contactref element="S2" pad="3"/>
+<contactref element="SW2" pad="4"/>
+<contactref element="SW2" pad="3"/>
 <contactref element="R2" pad="1"/>
 <wire x1="44.235" y1="20.955" x2="28.155" y2="20.955" width="0.254" layer="1"/>
@@
 <contactref element="U1" pad="5"/>
 <contactref element="R2" pad="2"/>
-<contactref element="S1" pad="4"/>
-<contactref element="S1" pad="3"/>
+<contactref element="SW1" pad="4"/>
+<contactref element="SW1" pad="3"/>
 <contactref element="R1" pad="1"/>
 <wire x1="26.455" y1="20.955" x2="10.375" y2="20.955" width="0.254" layer="1"/>
